Commit message: Adjust the origin of torso to mass center

File: urdf/fwmav_sjtu/flapper_sjtu.urdf (robot description, URDF)
Before this commit: robot flappy_sjtu, 7 links, 6 joints
Joints:
- joint servo_control: origin xyz=0.0 0.0 50E-3 rpy=0.0 0.0 0.0 -> xyz=1.286E-3 -0.551E-3 41.911E-3 rpy=0.0 0.0 0.0
